File: hw/bosonFrameGrabber_1_00/fileBoson.sch (KiCad schematic (older format))
At the start: 1 part, among them U5 Boson

Commit message: Update PCB with new footprint. Code project for bosonBreakout. (samd51) Simulation code for Verilog HyperRam module.
Parts:
- U5: PN (none) -> DF40HC(4.0)-80DS-0.4V(51); SN-DK (none) -> H11919CT-ND
Changed lines of the file:
@@
 EESchema Schematic File Version 4
+LIBS:bosonFrameGrabber-cache
 EELAYER 26 0
 EELAYER END
@@
 F 2 "" H 2100 4900 60  0001 C CNN
 F 3 "" H 2100 4900 60  0001 C CNN
+F 4 " H11919CT-ND " H 0   0   50  0001 C CNN "SN-DK"
+F 5 " DF40HC(4.0)-80DS-0.4V(51) " H 0   0   50  0001 C CNN "PN"
 	1    2100 3650
 	1    0    0    -1
@@
 F 2 "" H 5200 4500 60  0001 C CNN
 F 3 "" H 5200 4500 60  0001 C CNN
+F 4 " H11919CT-ND " H 0   0   50  0001 C CNN "SN-DK"
+F 5 " DF40HC(4.0)-80DS-0.4V(51) " H 0   0   50  0001 C CNN "PN"
 	2    5200 3250
 	1    0    0    -1
@@
 F 2 "" H 5050 7300 60  0001 C CNN
 F 3 "" H 5050 7300 60  0001 C CNN
+F 4 " H11919CT-ND " H 0   0   50  0001 C CNN "SN-DK"
+F 5 " DF40HC(4.0)-80DS-0.4V(51) " H 0   0   50  0001 C CNN "PN"
 	3    5050 6050
 	1    0    0    -1
@@
 F 2 "" H 8550 7000 60  0001 C CNN
 F 3 "" H 8550 7000 60  0001 C CNN
+F 4 " H11919CT-ND " H 0   0   50  0001 C CNN "SN-DK"
+F 5 " DF40HC(4.0)-80DS-0.4V(51) " H 0   0   50  0001 C CNN "PN"
 	4    8550 5750
 	1    0    0    -1
@@
 F 2 "" H 8450 3950 60  0001 C CNN
 F 3 "" H 8450 3950 60  0001 C CNN
+F 4 " H11919CT-ND " H 0   0   50  0001 C CNN "SN-DK"
+F 5 " DF40HC(4.0)-80DS-0.4V(51) " H 0   0   50  0001 C CNN "PN"
 	5    8450 2700
 	1    0    0    -1
