File: hw/bosonFrameGrabber_1_00/fileHyperRAM.sch (KiCad schematic (older format))
At the start: 2 parts, among them U4 S27KS0641, U6 AT25SF081

Commit message: Update PCB with new footprint. Code project for bosonBreakout. (samd51) Simulation code for Verilog HyperRam module.
Parts:
- U4: PN (none) -> S27KS0641DPBHI020; SN-DK (none) -> 428-3858-ND
- U6: PN (none) -> AT25SF081-MAHD-T; SN-DK (none) -> 1265-1275-1-ND
Changed lines of the file:
@@
 EESchema Schematic File Version 4
+LIBS:bosonFrameGrabber-cache
 EELAYER 26 0
 EELAYER END
@@
 F 2 "bosonFrameGrabber:BGA_24" H 7950 4850 60  0001 C CNN
 F 3 "" H 7950 4850 60  0001 C CNN
+F 4 " 428-3858-ND " H 0   0   50  0001 C CNN "SN-DK"
+F 5 "S27KS0641DPBHI020" H 0   0   50  0001 C CNN "PN"
 	1    7950 3900
 	1    0    0    -1
@@
 F 2 "Housings_DFN_QFN:DFN-8-1EP_3x2mm_Pitch0.5mm" H 4150 4400 60  0001 C CNN
 F 3 "" H 4150 4400 60  0001 C CNN
+F 4 " 1265-1275-1-ND " H 0   0   50  0001 C CNN "SN-DK"
+F 5 " AT25SF081-MAHD-T " H 0   0   50  0001 C CNN "PN"
 	1    4150 3950
 	1    0    0    -1
