File: hw/bosonFrameGrabber_1_00/fileIO.sch (KiCad schematic (older format))
At the start: 18 parts, among them J1 JST GH Series, U1 MIC5370, U2 SN74LVC1T45, U7 SN74LVC1T45

Commit message: Update PCB with new footprint. Code project for bosonBreakout. (samd51) Simulation code for Verilog HyperRam module.
Parts:
- C1, C2: PN (none) -> C0402C101J3GACTU; SN-DK (none) -> 399-1022-1-ND
- C13, C6, C7: PN (none) -> C1608X5R1A106K080AC; SN-DK (none) -> 445-7486-1-ND
- C3, C4: PN (none) -> CGB2A1X5R1E105K033BC; SN-DK (none) -> 445-13185-1-ND
- C5: value 100nF -> 100n; PN (none) -> CL05B104KP5NNNC; SN-DK (none) -> 1276-1002-1-ND
- D1: PN (none) -> LTST-C191KGKT; SN-DK (none) -> 160-1446-1-ND
- D2: PN (none) -> PESD5V0U2BT,215; SN-DK (none) -> 1727-3936-1-ND
- D3: PN (none) -> 1N4148X-TP; SN-DK (none) -> 1N4148XTPMSCT-ND
- J1: PN (none) -> BM05B-GHS-TBT(LF)(SN)(N); SN-DK (none) -> 455-1581-1-ND
- R1, R2: PN (none) -> RT0402FRE07100RL; SN-DK (none) -> YAG3342CT-ND
- R3: value R -> 470R; PN (none) -> RMCF0402JT470R; SN-DK (none) -> RMCF0402JT470RCT-ND
- U1: PN (none) -> MIC5370-G4YMT-TR; SN-DK (none) -> 576-3329-1-ND; SN-MO (none) -> 998-MIC5370-G4YMTTR
- U2, U7: PN (none) -> SN74LVC1T45DRLR; SN-DK (none) -> 296-20629-1-ND
Changed lines of the file:
@@
 EESchema Schematic File Version 4
+LIBS:bosonFrameGrabber-cache
 EELAYER 26 0
 EELAYER END
@@
 F 2 "LEDs:LED_0603" H 9100 2400 50  0001 C CNN
 F 3 "" H 9100 2400 50  0001 C CNN
+F 4 " 160-1446-1-ND " H 0   0   50  0001 C CNN "SN-DK"
+F 5 " LTST-C191KGKT " H 0   0   50  0001 C CNN "PN"
 	1    9100 2400
 	-1   0    0    1
@@
 P 9650 2400
 F 0 "R3" V 9443 2400 50  0000 C CNN
-F 1 "R" V 9534 2400 50  0000 C CNN
+F 1 "470R" V 9534 2400 50  0000 C CNN
 F 2 "Resistors_SMD:R_0402" V 9580 2400 50  0001 C CNN
 F 3 "" H 9650 2400 50  0001 C CNN
+F 4 " RMCF0402JT470RCT-ND " H 0   0   50  0001 C CNN "SN-DK"
+F 5 " RMCF0402JT470R " H 0   0   50  0001 C CNN "PN"
 	1    9650 2400
 	0    1    1    0
@@
 F 2 "Connectors_JST:JST_GH_BM06B-GHS-TBT_06x1.25mm_Straight" H 7200 2200 50  0001 C CNN
 F 3 "~" H 7200 2200 50  0001 C CNN
+F 4 " 455-1581-1-ND " H 0   0   50  0001 C CNN "SN-DK"
+F 5 " BM05B-GHS-TBT(LF)(SN)(N) " H 0   0   50  0001 C CNN "PN"
 	1    7200 2200
 	-1   0    0    -1
@@
 	7000 2100 6400 2100
 Wire Wire Line
-	6400 2100 6400 2650
+	6400 2100 6400 2300
 Text GLabel 7000 2400 0    60   Input ~ 0
 IO_A
@@
 F 2 "Resistors_SMD:R_0402" V 4980 1900 50  0001 C CNN
 F 3 "" H 5050 1900 50  0001 C CNN
+F 4 " YAG3342CT-ND " H 0   0   50  0001 C CNN "SN-DK"
+F 5 " RT0402FRE07100RL " H 0   0   50  0001 C CNN "PN"
 	1    5050 1900
 	0    1    1    0
@@
 F 2 "Resistors_SMD:R_0402" V 4980 2850 50  0001 C CNN
 F 3 "" H 5050 2850 50  0001 C CNN
+F 4 " YAG3342CT-ND " H 0   0   50  0001 C CNN "SN-DK"
+F 5 " RT0402FRE07100RL " H 0   0   50  0001 C CNN "PN"
 	1    5050 2850
 	0    1    1    0
 $EndComp
 Wire Wire Line
-	5200 1900 5550 1900
-Wire Wire Line
-	5200 2850 5550 2850
+	5200 1900 5350 1900
+Wire Wire Line
+	5200 2850 5350 2850
 $Comp
 L bosonFrameGrabber:SN74LVC1T45 U7
@@
 F 2 "TO_SOT_Packages_SMD:SOT-666" H 3900 2450 60  0001 C CNN
 F 3 "" H 3900 2450 60  0001 C CNN
+F 4 " 296-20629-1-ND " H 0   0   50  0001 C CNN "SN-DK"
+F 5 " SN74LVC1T45DRLR " H 0   0   50  0001 C CNN "PN"
 	1    3900 2450
 	1    0    0    -1
@@
 F 2 "TO_SOT_Packages_SMD:SOT-666" H 3900 1500 60  0001 C CNN
 F 3 "" H 3900 1500 60  0001 C CNN
+F 4 " 296-20629-1-ND " H 0   0   50  0001 C CNN "SN-DK"
+F 5 " SN74LVC1T45DRLR " H 0   0   50  0001 C CNN "PN"
 	1    3900 1500
 	1    0    0    -1
@@
 $EndComp
 Wire Wire Line
-	4350 1900 4900 1900
-Wire Wire Line
-	4350 2850 4900 2850
+	4350 1900 4800 1900
+Wire Wire Line
+	4350 2850 4800 2850
 Wire Wire Line
 	3200 1900 3450 1900
@@
 	3450 1800 3350 1800
 Wire Wire Line
-	3350 1800 3350 3200
+	3350 1800 3350 2750
 $Comp
 L bosonFrameGrabber:+3V3 #PWR07
@@
 	3450 1700 3250 1700
 Wire Wire Line
-	3250 1550 3250 2650
+	3250 1550 3250 1700
 Wire Wire Line
 	3450 2650 3250 2650
@@
 $EndComp
 Wire Wire Line
-	4550 1550 4550 2650
+	4550 1550 4550 1700
 Wire Wire Line
 	4550 2650 4350 2650
@@
 F 2 "Capacitors_SMD:C_0402" H 4838 2050 50  0001 C CNN
 F 3 "" H 4800 2200 50  0001 C CNN
+F 4 " 399-1022-1-ND " H 0   0   50  0001 C CNN "SN-DK"
+F 5 "C0402C101J3GACTU" H 0   0   50  0001 C CNN "PN"
 	1    4800 2200
 	1    0    0    -1
@@
 F 2 "Capacitors_SMD:C_0402" H 4838 3000 50  0001 C CNN
 F 3 "" H 4800 3150 50  0001 C CNN
+F 4 " 399-1022-1-ND " H 0   0   50  0001 C CNN "SN-DK"
+F 5 "C0402C101J3GACTU" H 0   0   50  0001 C CNN "PN"
 	1    4800 3150
 	1    0    0    -1
@@
 F 2 "TO_SOT_Packages_SMD:SOT-23" H 5200 2400 50  0001 C CNN
 F 3 "https://en.wikipedia.org/wiki/Transient-voltage-suppression_diode" H 5200 2400 50  0001 C CNN
+F 4 " 1727-3936-1-ND " H 0   0   50  0001 C CNN "SN-DK"
+F 5 " PESD5V0U2BT,215 " H 0   0   50  0001 C CNN "PN"
 	1    5350 2400
 	0    -1   -1   0
@@
 F 2 "" H 3850 5850 60  0001 C CNN
 F 3 "" H 3850 5850 60  0001 C CNN
+F 4 " 576-3329-1-ND " H 0   0   50  0001 C CNN "SN-DK"
+F 5 " MIC5370-G4YMT-TR " H 0   0   50  0001 C CNN "PN"
+F 6 " 998-MIC5370-G4YMTTR " H 0   0   50  0001 C CNN "SN-MO"
 	1    3850 5450
 	1    0    0    -1
@@
 F 2 "Capacitors_SMD:C_0402" H 4838 5750 50  0001 C CNN
 F 3 "" H 4800 5900 50  0001 C CNN
+F 4 " 445-13185-1-ND " H 0   0   50  0001 C CNN "SN-DK"
+F 5 "CGB2A1X5R1E105K033BC" H 0   0   50  0001 C CNN "PN"
 	1    4800 5900
 	1    0    0    -1
@@
 F 2 "Capacitors_SMD:C_0402" H 5288 5750 50  0001 C CNN
 F 3 "" H 5250 5900 50  0001 C CNN
+F 4 " 445-13185-1-ND " H 0   0   50  0001 C CNN "SN-DK"
+F 5 "CGB2A1X5R1E105K033BC" H 0   0   50  0001 C CNN "PN"
 	1    5250 5900
 	1    0    0    -1
@@
 	4350 5300 5250 5300
 Wire Wire Line
-	5250 5100 5250 5750
+	5250 5100 5250 5300
 Wire Wire Line
 	4350 5600 4800 5600
 Wire Wire Line
-	4800 5100 4800 5750
+	4800 5100 4800 5600
 Wire Wire Line
 	3350 5800 3200 5800
 Wire Wire Line
-	3200 5800 3200 6150
+	3200 5800 3200 5900
 Wire Wire Line
 	3350 5900 3200 5900
@@
 	3350 5600 3200 5600
 Wire Wire Line
-	3200 5600 3200 5100
+	3200 5600 3200 5500
 Wire Wire Line
 	3350 5300 3200 5300
@@
 F 2 "Diodes_SMD:D_SC-80" H 6100 5250 50  0001 C CNN
 F 3 "" H 6100 5250 50  0001 C CNN
+F 4 " 1N4148XTPMSCT-ND " H 0   0   50  0001 C CNN "SN-DK"
+F 5 " 1N4148X-TP " H 0   0   50  0001 C CNN "PN"
 	1    6100 5250
 	-1   0    0    1
@@
 P 6400 5550
 F 0 "C5" H 6515 5596 50  0000 L CNN
-F 1 "100nF" H 6515 5505 50  0000 L CNN
+F 1 "100n" H 6515 5505 50  0000 L CNN
 F 2 "Capacitors_SMD:C_0402" H 6438 5400 50  0001 C CNN
 F 3 "" H 6400 5550 50  0001 C CNN
+F 4 " 1276-1002-1-ND " H 0   0   50  0001 C CNN "SN-DK"
+F 5 " CL05B104KP5NNNC " H 0   0   50  0001 C CNN "PN"
 	1    6400 5550
 	1    0    0    -1
@@
 	6250 5250 6400 5250
 Wire Wire Line
-	6400 5100 6400 5400
+	6400 5100 6400 5250
 Connection ~ 6400 5250
 Wire Wire Line
@@
 F 2 "Capacitors_SMD:C_0603" H 2088 5450 50  0001 C CNN
 F 3 "" H 2050 5600 50  0001 C CNN
+F 4 " 445-7486-1-ND " H 0   0   50  0001 C CNN "SN-DK"
+F 5 "C1608X5R1A106K080AC" H 0   0   50  0001 C CNN "PN"
 	1    2050 5600
 	1    0    0    -1
@@
 F 2 "Capacitors_SMD:C_0603" H 2488 5450 50  0001 C CNN
 F 3 "" H 2450 5600 50  0001 C CNN
+F 4 " 445-7486-1-ND " H 0   0   50  0001 C CNN "SN-DK"
+F 5 "C1608X5R1A106K080AC" H 0   0   50  0001 C CNN "PN"
 	1    2450 5600
 	1    0    0    -1
@@
 F 2 "Capacitors_SMD:C_0603" H 1688 5450 50  0001 C CNN
 F 3 "" H 1650 5600 50  0001 C CNN
+F 4 " 445-7486-1-ND " H 0   0   50  0001 C CNN "SN-DK"
+F 5 "C1608X5R1A106K080AC" H 0   0   50  0001 C CNN "PN"
 	1    1650 5600
 	1    0    0    -1
@@
 	1    0    0    -1
 $EndComp
+Wire Wire Line
+	6400 2300 6400 2500
+Wire Wire Line
+	6400 2500 6400 2650
+Wire Wire Line
+	3250 1700 3250 2650
+Wire Wire Line
+	3350 2750 3350 3200
+Wire Wire Line
+	4550 1700 4550 2650
+Wire Wire Line
+	4800 2850 4900 2850
+Wire Wire Line
+	4800 1900 4900 1900
+Wire Wire Line
+	5350 2850 5550 2850
+Wire Wire Line
+	5350 1900 5550 1900
+Wire Wire Line
+	3200 5900 3200 6150
+Wire Wire Line
+	3200 5300 3200 5100
+Wire Wire Line
+	3200 5500 3200 5300
+Wire Wire Line
+	4800 5600 4800 5750
+Wire Wire Line
+	5250 5300 5250 5750
+Wire Wire Line
+	6400 5250 6400 5400
 $EndSCHEMATC
