File: hw/bosonFrameGrabber_1_00/fileSDMMC.sch (KiCad schematic (older format))
At the start: 1 part, among them J4 MicroSD

Commit message: Update PCB with new footprint. Code project for bosonBreakout. (samd51) Simulation code for Verilog HyperRam module.
Parts:
- J4: PN (none) -> 1040310811
Changed lines of the file:
@@
 EESchema Schematic File Version 4
+LIBS:bosonFrameGrabber-cache
 EELAYER 26 0
 EELAYER END
@@
 F 3 "~" H 5650 3850 50  0001 C CNN
 F 4 " WM6357CT-ND" H 5650 3850 60  0001 C CNN "SN-DK"
+F 5 "1040310811" H 0   0   50  0001 C CNN "PN"
 	1    5650 3850
 	-1   0    0    -1
