File: hw/bosonFrameGrabber_1_02/bosonFrameGrabber.kicad_pcb (KiCad board)
At the start: 4 copper layers, 21 x 21 mm, 48 parts, among them J1 JST GH Series, J4 MicroSD, U1 TLV733P, U2 SN74LVC1T45, U3 ECP5U25, U4 S27KS0641, U5 Boson, U6 AT25SF081, U7 SN74LVC1T45, U8 TLV733P, U9 TLV733P, X1 ASDMB

Commit message: Updates to project documentation.
Parts:
- R3: value R -> 10k
- U1: value TLV733P -> TLV70725
- U8: value TLV733P -> TLV71718
- U9: value TLV733P -> TLV73311
