File: hw/bosonFrameGrabber_1_02/fileFPGA.sch (KiCad schematic (older format))
At the start: 3 parts, among them U3 ECP5U25, X1 ASDMB

Commit message: Updates to project documentation.
Parts:
- U3: PN (none) -> LFE5UM-25F-6MG285C; SN-DK (none) -> LFE5UM-25F-6MG285C-ND
- X1: PN (none) -> SIT8008BI-71-18E-24.000000G; SN-DK (none) -> 1473-30509-1-ND
Changed lines of the file:
@@
 F 2 "Oscillators:Oscillator_SMD_SeikoEpson_SG210-4pin_2.5x2.0mm" H 8450 5150 50  0001 C CNN
 F 3 "http://www.abracon.com/Oscillators/ASV.pdf" H 7650 5500 50  0001 C CNN
+F 4 "SIT8008BI-71-18E-24.000000G" H 0   0   50  0001 C CNN "PN"
+F 5 "1473-30509-1-ND" H 0   0   50  0001 C CNN "SN-DK"
 	1    7750 5500
 	1    0    0    -1
@@
 F 2 "" H 2550 1100 50  0001 C CNN
 F 3 "" H 2550 1100 50  0001 C CNN
+F 4 "LFE5UM-25F-6MG285C " H 0   0   50  0001 C CNN "PN"
+F 5 " LFE5UM-25F-6MG285C-ND " H 0   0   50  0001 C CNN "SN-DK"
 	1    2550 1100
 	-1   0    0    -1
@@
 F 2 "" H 2550 2200 50  0001 C CNN
 F 3 "" H 2550 2200 50  0001 C CNN
+F 4 "LFE5UM-25F-6MG285C " H 0   0   50  0001 C CNN "PN"
+F 5 " LFE5UM-25F-6MG285C-ND " H 0   0   50  0001 C CNN "SN-DK"
 	2    2550 2200
 	-1   0    0    -1
@@
 F 2 "" H 2550 3250 50  0001 C CNN
 F 3 "" H 2550 3250 50  0001 C CNN
+F 4 "LFE5UM-25F-6MG285C " H 0   0   50  0001 C CNN "PN"
+F 5 " LFE5UM-25F-6MG285C-ND " H 0   0   50  0001 C CNN "SN-DK"
 	3    2550 3250
 	-1   0    0    -1
@@
 F 2 "" H 5650 1250 50  0001 C CNN
 F 3 "" H 5650 1250 50  0001 C CNN
+F 4 "LFE5UM-25F-6MG285C " H 0   0   50  0001 C CNN "PN"
+F 5 " LFE5UM-25F-6MG285C-ND " H 0   0   50  0001 C CNN "SN-DK"
 	4    5650 1250
 	-1   0    0    -1
@@
 F 2 "" H 5650 4950 50  0001 C CNN
 F 3 "" H 5650 4950 50  0001 C CNN
+F 4 "LFE5UM-25F-6MG285C " H 0   0   50  0001 C CNN "PN"
+F 5 " LFE5UM-25F-6MG285C-ND " H 0   0   50  0001 C CNN "SN-DK"
 	5    5650 4950
 	-1   0    0    -1
@@
 F 2 "" H 2550 5750 50  0001 C CNN
 F 3 "" H 2550 5750 50  0001 C CNN
+F 4 "LFE5UM-25F-6MG285C " H 0   0   50  0001 C CNN "PN"
+F 5 " LFE5UM-25F-6MG285C-ND " H 0   0   50  0001 C CNN "SN-DK"
 	6    2550 5750
 	-1   0    0    -1
@@
 F 2 "" H 9250 1250 50  0001 C CNN
 F 3 "" H 9250 1250 50  0001 C CNN
+F 4 "LFE5UM-25F-6MG285C " H 0   0   50  0001 C CNN "PN"
+F 5 " LFE5UM-25F-6MG285C-ND " H 0   0   50  0001 C CNN "SN-DK"
 	7    9250 1250
 	-1   0    0    -1
@@
 F 2 "" H 9250 2900 50  0001 C CNN
 F 3 "" H 9250 2900 50  0001 C CNN
+F 4 "LFE5UM-25F-6MG285C " H 0   0   50  0001 C CNN "PN"
+F 5 " LFE5UM-25F-6MG285C-ND " H 0   0   50  0001 C CNN "SN-DK"
 	8    9250 2900
 	-1   0    0    -1
@@
 F 2 "" H 9850 5900 50  0001 C CNN
 F 3 "" H 9850 5900 50  0001 C CNN
+F 4 "LFE5UM-25F-6MG285C " H 0   0   50  0001 C CNN "PN"
+F 5 " LFE5UM-25F-6MG285C-ND " H 0   0   50  0001 C CNN "SN-DK"
 	9    9850 5900
 	1    0    0    1
