File: hw/bosonFrameGrabber_1_02/fileIO.sch (KiCad schematic (older format))
At the start: 33 parts, among them J1 JST GH Series, U1 TLV733P, U2 SN74LVC1T45, U7 SN74LVC1T45, U8 TLV733P, U9 TLV733P

Commit message: Updates to project documentation.
Parts:
- D1: PN (none) -> APHHS1005SYCK; SN-DK (none) -> 754-1105-1-ND
- J1: PN (none) -> BM06B-GHS-TBT(LF)(SN)(N); SN-DK (none) -> 455-1582-1-ND
- U1: value TLV733P -> TLV70725; PN (none) -> TLV70725PDQNT; SN-DK (none) -> 296-34993-1-ND
- U8: value TLV733P -> TLV71718; PN (none) -> TLV71718PDQNR; SN-DK (none) -> 296-36775-1-ND
- U9: value TLV733P -> TLV73311; PN (none) -> TLV73311PDQNT; SN-DK (none) -> 296-38619-1-ND
Changed lines of the file:
@@
 F 2 "LEDs:LED_0603" H 8750 1950 50  0001 C CNN
 F 3 "" H 8750 1950 50  0001 C CNN
+F 4 "APHHS1005SYCK " H 0   0   50  0001 C CNN "PN"
+F 5 "754-1105-1-ND" H 0   0   50  0001 C CNN "SN-DK"
 	1    8750 1950
 	-1   0    0    1
@@
 F 2 "Connectors_JST:JST_GH_BM06B-GHS-TBT_06x1.25mm_Straight" H 6800 1900 50  0001 C CNN
 F 3 "~" H 6800 1900 50  0001 C CNN
+F 4 "BM06B-GHS-TBT(LF)(SN)(N) " H 0   0   50  0001 C CNN "PN"
+F 5 "455-1582-1-ND" H 0   0   50  0001 C CNN "SN-DK"
 	1    6800 1900
 	-1   0    0    -1
@@
 P 2750 5350
 F 0 "U1" H 2750 5675 50  0000 C CNN
-F 1 "TLV733P" H 2750 5584 50  0000 C CNN
+F 1 "TLV70725" H 2750 5584 50  0000 C CNN
 F 2 "bosonFrameGrabber:X2SON" H 2750 5600 50  0001 C CNN
 F 3 "" H 2750 5600 50  0001 C CNN
+F 4 "TLV70725PDQNT " H 0   0   50  0001 C CNN "PN"
+F 5 "296-34993-1-ND" H 0   0   50  0001 C CNN "SN-DK"
 	1    2750 5350
 	1    0    0    -1
@@
 P 2750 6100
 F 0 "U8" H 2750 6425 50  0000 C CNN
-F 1 "TLV733P" H 2750 6334 50  0000 C CNN
+F 1 "TLV71718" H 2750 6334 50  0000 C CNN
 F 2 "bosonFrameGrabber:X2SON" H 2750 6350 50  0001 C CNN
 F 3 "" H 2750 6350 50  0001 C CNN
+F 4 "TLV71718PDQNR " H 0   0   50  0001 C CNN "PN"
+F 5 "296-36775-1-ND" H 0   0   50  0001 C CNN "SN-DK"
 	1    2750 6100
 	1    0    0    -1
@@
 P 2750 6850
 F 0 "U9" H 2750 7175 50  0000 C CNN
-F 1 "TLV733P" H 2750 7084 50  0000 C CNN
+F 1 "TLV73311" H 2750 7084 50  0000 C CNN
 F 2 "bosonFrameGrabber:X2SON" H 2750 7100 50  0001 C CNN
 F 3 "" H 2750 7100 50  0001 C CNN
+F 4 "TLV73311PDQNT " H 0   0   50  0001 C CNN "PN"
+F 5 "296-38619-1-ND" H 0   0   50  0001 C CNN "SN-DK"
 	1    2750 6850
 	1    0    0    -1
